File: kicad/adressInverter.kicad_sch (KiCad schematic)
At the start: 2 parts, among them U1 74LS86

Commit message: finished footprints and started layout
Parts:
- C1: footprint (none) -> Capacitor_THT:C_Disc_D3.0mm_W1.6mm_P2.50mm
Changed lines of the file:
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@@
       (effects (font (size 1.27 1.27)) (justify left))
     )
-    (property "Footprint" "" (at 134.3152 130.81 0)
+    (property "Footprint" "Capacitor_THT:C_Disc_D3.0mm_W1.6mm_P2.50mm" (at 134.3152 130.81 0)
       (effects (font (size 1.27 1.27)) hide)
     )
