File: kicad/com_dmuxUP.kicad_sch (KiCad schematic)
At the start: 10 parts, among them U1 7421, U3 74LS138, U4 7421, U5 7421, U6 74LS138

Commit message: finished footprints and started layout
Parts:
- C1, C3, C4, C5, C6: footprint (none) -> Capacitor_THT:C_Disc_D3.0mm_W1.6mm_P2.50mm
- U1, U4, U5: footprint (none) -> Package_DIP:DIP-14_W10.16mm_LongPads
- U3, U6: footprint (none) -> Package_DIP:DIP-16_W10.16mm_LongPads
Changed lines of the file:
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@@
       (effects (font (size 1.27 1.27)))
     )
-    (property "Footprint" "" (at 381 152.4 0)
+    (property "Footprint" "Package_DIP:DIP-14_W10.16mm_LongPads" (at 381 152.4 0)
       (effects (font (size 1.27 1.27)) hide)
     )
@@
       (effects (font (size 1.27 1.27)) (justify left))
     )
-    (property "Footprint" "" (at 234.6452 325.12 0)
+    (property "Footprint" "Capacitor_THT:C_Disc_D3.0mm_W1.6mm_P2.50mm" (at 234.6452 325.12 0)
       (effects (font (size 1.27 1.27)) hide)
     )
@@
       (effects (font (size 1.27 1.27)) (justify left))
     )
-    (property "Footprint" "" (at 287.02 269.24 0)
+    (property "Footprint" "Package_DIP:DIP-16_W10.16mm_LongPads" (at 287.02 269.24 0)
       (effects (font (size 1.27 1.27)) hide)
     )
@@
       (effects (font (size 1.27 1.27)))
     )
-    (property "Footprint" "" (at 381 233.68 0)
+    (property "Footprint" "Package_DIP:DIP-14_W10.16mm_LongPads" (at 381 233.68 0)
       (effects (font (size 1.27 1.27)) hide)
     )
@@
       (effects (font (size 1.27 1.27)) (justify left))
     )
-    (property "Footprint" "" (at 228.2952 325.12 0)
+    (property "Footprint" "Capacitor_THT:C_Disc_D3.0mm_W1.6mm_P2.50mm" (at 228.2952 325.12 0)
       (effects (font (size 1.27 1.27)) hide)
     )
@@
       (effects (font (size 1.27 1.27)) (justify left))
     )
-    (property "Footprint" "" (at 287.02 148.59 0)
+    (property "Footprint" "Package_DIP:DIP-16_W10.16mm_LongPads" (at 287.02 148.59 0)
       (effects (font (size 1.27 1.27)) hide)
     )
@@
       (effects (font (size 1.27 1.27)) (justify left))
     )
-    (property "Footprint" "" (at 253.6952 325.12 0)
+    (property "Footprint" "Capacitor_THT:C_Disc_D3.0mm_W1.6mm_P2.50mm" (at 253.6952 325.12 0)
       (effects (font (size 1.27 1.27)) hide)
     )
@@
       (effects (font (size 1.27 1.27)))
     )
-    (property "Footprint" "" (at 381 111.76 0)
+    (property "Footprint" "Package_DIP:DIP-14_W10.16mm_LongPads" (at 381 111.76 0)
       (effects (font (size 1.27 1.27)) hide)
     )
@@
       (effects (font (size 1.27 1.27)) (justify left))
     )
-    (property "Footprint" "" (at 247.3452 325.12 0)
+    (property "Footprint" "Capacitor_THT:C_Disc_D3.0mm_W1.6mm_P2.50mm" (at 247.3452 325.12 0)
       (effects (font (size 1.27 1.27)) hide)
     )
@@
       (effects (font (size 1.27 1.27)) (justify left))
     )
-    (property "Footprint" "" (at 240.9952 325.12 0)
+    (property "Footprint" "Capacitor_THT:C_Disc_D3.0mm_W1.6mm_P2.50mm" (at 240.9952 325.12 0)
       (effects (font (size 1.27 1.27)) hide)
     )
@@
       (effects (font (size 1.27 1.27)))
     )
-    (property "Footprint" "" (at 381 274.32 0)
+    (property "Footprint" "Package_DIP:DIP-14_W10.16mm_LongPads" (at 381 274.32 0)
       (effects (font (size 1.27 1.27)) hide)
     )
@@
       (effects (font (size 1.27 1.27)))
     )
-    (property "Footprint" "" (at 381 314.96 0)
+    (property "Footprint" "Package_DIP:DIP-14_W10.16mm_LongPads" (at 381 314.96 0)
       (effects (font (size 1.27 1.27)) hide)
     )
@@
       (effects (font (size 1.27 1.27)))
     )
-    (property "Footprint" "" (at 381 193.04 0)
-      (effects (font (size 1.27 1.27)) hide)
-    )
+    (property "Footprint" "Package_DIP:DIP-14_W10.16mm_LongPads" (at 381 193.04 0)
+      (effects (font (size 1.27 1.27)) hide)
+    )
