File: kicad/main.kicad_sch (KiCad schematic)
At the start: 0 parts

Commit message: added schematic for demux
Parts:
- added J1: Conn_02x14_Counter_Clockwise, symbol Connector_Generic:Conn_02x14_Counter_Clockwise
Connections:
- new net +5V: J1.28 (Pin_28)
- new net B_H_OUT: J1.11 (Pin_11)
- new net B_L_OUT: J1.15 (Pin_15)
- new net DIR_IN: J1.7 (Pin_7)
- new net GND: J1.14 (Pin_14)
- new net G_H_OUT: J1.12 (Pin_12)
- new net G_L_OUT: J1.16 (Pin_16)
- new net H1_IN: J1.10 (Pin_10)
- new net H2_IN: J1.9 (Pin_9)
- new net H3_IN: J1.8 (Pin_8)
- new net PWM_IN: J1.6 (Pin_6)
- new net Y_H_OUT: J1.13 (Pin_13)
- new net Y_L_OUT: J1.17 (Pin_17)
- no-connect marks 0 -> 15
Other:
- added sheet adressInverter (adressInverter.kicad_sch)
- added sheet com_dmux (com_dmuxUP.kicad_sch)

Commit message: finished footprints and started layout
Parts:
- J1: footprint (none) -> Package_DIP:DIP-28_W15.24mm_Socket_LongPads
Changed lines of the file:
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@@
       (effects (font (size 1.27 1.27)))
     )
-    (property "Footprint" "" (at 50.8 132.08 0)
+    (property "Footprint" "Package_DIP:DIP-28_W15.24mm_Socket_LongPads" (at 50.8 132.08 0)
       (effects (font (size 1.27 1.27)) hide)
     )
